Commit message: [Sim] Figured out the sensors freeze problem

File: urdf/materials.xacro (robot description, xacro)
@@ -1,6 +1,2 @@
-<?xml version="1.0" ?>
-<robot name="sim" xmlns:xacro="http://www.ros.org/wiki/xacro" >
-<material name="silver">
-  <color rgba="0.700 0.700 0.700 1.000"/>
-</material>
-</robot>
+<?xml version='1.0' encoding='utf-8'?>
+<robot name="sim" xmlns:xacro="http://www.ros.org/wiki/xacro"><material name="fusion_Nylon_12__with_Formlabs_Fuse_1_3D_Printer__9b6938a61d"><color rgba="0.24705882 0.24705882 0.24705882 1" /></material><material name="fusion_Steel___Satin_7dcf9b04aa"><color rgba="0.62352941 0.62352941 0.62352941 1" /></material><material name="fusion_Plastic___Glossy__Black__77387cc1bc"><color rgba="0.098039216 0.098039216 0.098039216 0" /></material><material name="fusion_Paek__Beige__c3b53efd9f"><color rgba="0.97647059 0.6745098 0.18431373 1" /></material><material name="fusion_Plastic___Glossy__Black__e2e6ed1680"><color rgba="0.098039216 0.098039216 0.098039216 1" /></material></robot>

File: urdf/sim.xacro (robot description, xacro)
@@ -10,10 +10,10 @@
     <inertia ixx="0.032507" iyy="0.034335" izz="0.029521" ixy="-0.0" iyz="0.001867" ixz="0.0"/>
   </inertial>
-  <visual>
+  <visual name="visual_0">
     <origin xyz="0 0 0" rpy="0 0 0"/>
     <geometry>
-      <mesh filename="file://$(find sim_description)/meshes/base_link.stl" scale="0.001 0.001 0.001"/>
-    </geometry>
-    <material name="silver"/>
+      <mesh filename="file://$(find sim_description)/meshes/__visual__base_link_715a4d03a5_0.stl" scale="0.001 0.001 0.001"/>
+    </geometry>
+    <material name="fusion_Paek__Beige__c3b53efd9f"/>
   </visual>
   <collision>
@@ -30,10 +30,10 @@
     <inertia ixx="4e-06" iyy="0.0" izz="4e-06" ixy="-0.0" iyz="-0.0" ixz="-0.0"/>
   </inertial>
-  <visual>
+  <visual name="visual_0">
     <origin xyz="-0.27 0.012358 -0.2" rpy="0 0 0"/>
     <geometry>
-      <mesh filename="file://$(find sim_description)/meshes/Button_Head_Small_Solid_Rivet_ASME_B18.1.1_-_3_8_x_1_1_4_Steel_Plain_1.stl" scale="0.001 0.001 0.001"/>
-    </geometry>
-    <material name="silver"/>
+      <mesh filename="file://$(find sim_description)/meshes/__visual__Button_Head_Small_Solid_Rivet_ASME_B18.1.1_-_3_8_x_1_1_4_Steel_Plain_1_053bc43f51_0.stl" scale="0.001 0.001 0.001"/>
+    </geometry>
+    <material name="fusion_Steel___Satin_7dcf9b04aa"/>
   </visual>
   <collision>
@@ -50,10 +50,10 @@
     <inertia ixx="6.8e-05" iyy="4e-05" izz="4e-05" ixy="0.0" iyz="-0.0" ixz="0.0"/>
   </inertial>
-  <visual>
+  <visual name="visual_0">
     <origin xyz="-0.665 0.042358 -0.017023" rpy="0 0 0"/>
     <geometry>
-      <mesh filename="file://$(find sim_description)/meshes/Wheel2_1.stl" scale="0.001 0.001 0.001"/>
-    </geometry>
-    <material name="silver"/>
+      <mesh filename="file://$(find sim_description)/meshes/__visual__Wheel2_1_6cc1698ccd_0.stl" scale="0.001 0.001 0.001"/>
+    </geometry>
+    <material name="fusion_Nylon_12__with_Formlabs_Fuse_1_3D_Printer__9b6938a61d"/>
   </visual>
   <collision>
@@ -70,10 +70,10 @@
     <inertia ixx="6.8e-05" iyy="4e-05" izz="4e-05" ixy="0.0" iyz="-0.0" ixz="0.0"/>
   </inertial>
-  <visual>
+  <visual name="visual_0">
     <origin xyz="-0.665 -0.057642 -0.017023" rpy="0 0 0"/>
     <geometry>
-      <mesh filename="file://$(find sim_description)/meshes/Wheels_1.stl" scale="0.001 0.001 0.001"/>
-    </geometry>
-    <material name="silver"/>
+      <mesh filename="file://$(find sim_description)/meshes/__visual__Wheels_1_594b391ede_0.stl" scale="0.001 0.001 0.001"/>
+    </geometry>
+    <material name="fusion_Nylon_12__with_Formlabs_Fuse_1_3D_Printer__9b6938a61d"/>
   </visual>
   <collision>
@@ -90,10 +90,10 @@
     <inertia ixx="6.8e-05" iyy="4e-05" izz="4e-05" ixy="0.0" iyz="-0.0" ixz="0.0"/>
   </inertial>
-  <visual>
+  <visual name="visual_0">
     <origin xyz="-0.415 0.042358 -0.017023" rpy="0 0 0"/>
     <geometry>
-      <mesh filename="file://$(find sim_description)/meshes/Wheels3_1.stl" scale="0.001 0.001 0.001"/>
-    </geometry>
-    <material name="silver"/>
+      <mesh filename="file://$(find sim_description)/meshes/__visual__Wheels3_1_788b86b6ca_0.stl" scale="0.001 0.001 0.001"/>
+    </geometry>
+    <material name="fusion_Nylon_12__with_Formlabs_Fuse_1_3D_Printer__9b6938a61d"/>
   </visual>
   <collision>
@@ -110,10 +110,10 @@
     <inertia ixx="6.8e-05" iyy="4e-05" izz="4e-05" ixy="0.0" iyz="-0.0" ixz="0.0"/>
   </inertial>
-  <visual>
+  <visual name="visual_0">
     <origin xyz="-0.415 -0.057642 -0.017023" rpy="0 0 0"/>
     <geometry>
-      <mesh filename="file://$(find sim_description)/meshes/Wheels4_1.stl" scale="0.001 0.001 0.001"/>
-    </geometry>
-    <material name="silver"/>
+      <mesh filename="file://$(find sim_description)/meshes/__visual__Wheels4_1_2e6ca671c6_0.stl" scale="0.001 0.001 0.001"/>
+    </geometry>
+    <material name="fusion_Nylon_12__with_Formlabs_Fuse_1_3D_Printer__9b6938a61d"/>
   </visual>
   <collision>
@@ -130,10 +130,10 @@
     <inertia ixx="9.8e-05" iyy="3.1e-05" izz="6.8e-05" ixy="-0.0" iyz="-3.6e-05" ixz="0.0"/>
   </inertial>
-  <visual>
+  <visual name="visual_0">
     <origin xyz="-0.158 0.052358 -0.109854" rpy="0 0 0"/>
     <geometry>
-      <mesh filename="file://$(find sim_description)/meshes/Simple-Hand2_1.stl" scale="0.001 0.001 0.001"/>
-    </geometry>
-    <material name="silver"/>
+      <mesh filename="file://$(find sim_description)/meshes/__visual__Simple-Hand2_1_7b7cf8c415_0.stl" scale="0.001 0.001 0.001"/>
+    </geometry>
+    <material name="fusion_Nylon_12__with_Formlabs_Fuse_1_3D_Printer__9b6938a61d"/>
   </visual>
   <collision>
@@ -150,10 +150,10 @@
     <inertia ixx="9.8e-05" iyy="3.1e-05" izz="6.8e-05" ixy="0.0" iyz="-3.6e-05" ixz="-0.0"/>
   </inertial>
-  <visual>
+  <visual name="visual_0">
     <origin xyz="-0.382 0.052358 -0.109854" rpy="0 0 0"/>
     <geometry>
-      <mesh filename="file://$(find sim_description)/meshes/Simple-Hand_1.stl" scale="0.001 0.001 0.001"/>
-    </geometry>
-    <material name="silver"/>
+      <mesh filename="file://$(find sim_description)/meshes/__visual__Simple-Hand_1_5e8c8bbd99_0.stl" scale="0.001 0.001 0.001"/>
+    </geometry>
+    <material name="fusion_Nylon_12__with_Formlabs_Fuse_1_3D_Printer__9b6938a61d"/>
   </visual>
   <collision>
@@ -170,10 +170,10 @@
     <inertia ixx="0.000123" iyy="0.000121" izz="6e-06" ixy="0.0" iyz="-0.0" ixz="0.0"/>
   </inertial>
-  <visual>
+  <visual name="visual_0">
     <origin xyz="-0.27 0.007358 -0.2" rpy="0 0 0"/>
     <geometry>
-      <mesh filename="file://$(find sim_description)/meshes/Neck_1.stl" scale="0.001 0.001 0.001"/>
-    </geometry>
-    <material name="silver"/>
+      <mesh filename="file://$(find sim_description)/meshes/__visual__Neck_1_34c932d70d_0.stl" scale="0.001 0.001 0.001"/>
+    </geometry>
+    <material name="fusion_Nylon_12__with_Formlabs_Fuse_1_3D_Printer__9b6938a61d"/>
   </visual>
   <collision>
@@ -190,10 +190,10 @@
     <inertia ixx="0.000921" iyy="0.001304" izz="0.001096" ixy="-4e-06" iyz="-2e-06" ixz="-0.000273"/>
   </inertial>
-  <visual>
+  <visual name="visual_0">
     <origin xyz="-0.27 -0.007642 -0.349854" rpy="0 0 0"/>
     <geometry>
-      <mesh filename="file://$(find sim_description)/meshes/Eye-Piece_1.stl" scale="0.001 0.001 0.001"/>
-    </geometry>
-    <material name="silver"/>
+      <mesh filename="file://$(find sim_description)/meshes/__visual__Eye-Piece_1_6ef455a09f_0.stl" scale="0.001 0.001 0.001"/>
+    </geometry>
+    <material name="fusion_Nylon_12__with_Formlabs_Fuse_1_3D_Printer__9b6938a61d"/>
   </visual>
   <collision>
@@ -210,30 +210,30 @@
     <inertia ixx="0.000916" iyy="0.001291" izz="0.001087" ixy="-0.0" iyz="-0.0" ixz="0.000267"/>
   </inertial>
-  <visual>
+  <visual name="visual_0">
     <origin xyz="-0.27 0.002358 -0.349854" rpy="0 0 0"/>
     <geometry>
+      <mesh filename="file://$(find sim_description)/meshes/__visual__Eye-Piece_other_1_aa47e234cb_0.stl" scale="0.001 0.001 0.001"/>
+    </geometry>
+    <material name="fusion_Nylon_12__with_Formlabs_Fuse_1_3D_Printer__9b6938a61d"/>
+  </visual>
+  <collision>
+    <origin xyz="-0.27 0.002358 -0.349854" rpy="0 0 0"/>
+    <geometry>
       <mesh filename="file://$(find sim_description)/meshes/Eye-Piece_other_1.stl" scale="0.001 0.001 0.001"/>
     </geometry>
-    <material name="silver"/>
-  </visual>
-  <collision>
-    <origin xyz="-0.27 0.002358 -0.349854" rpy="0 0 0"/>
-    <geometry>
-      <mesh filename="file://$(find sim_description)/meshes/Eye-Piece_other_1.stl" scale="0.001 0.001 0.001"/>
-    </geometry>
   </collision>
 </link>
 <link name="eye_CAM_1">
   <inertial>
-    <origin xyz="-2.8683158786846352e-05 -0.002358818871701897 -0.00010604032573846567" rpy="0 0 0"/>
+    <origin xyz="-2.8683158786846352e-05 -0.00235881887170189 -0.0001060403257386322" rpy="0 0 0"/>
     <mass value="0.0026282548716325452"/>
     <inertia ixx="0.0" iyy="0.0" izz="0.0" ixy="-0.0" iyz="-0.0" ixz="0.0"/>
   </inertial>
-  <visual>
+  <visual name="visual_0">
     <origin xyz="-0.342218 0.032358 -0.302551" rpy="0 0 0"/>
     <geometry>
-      <mesh filename="file://$(find sim_description)/meshes/eye_CAM_1.stl" scale="0.001 0.001 0.001"/>
-    </geometry>
-    <material name="silver"/>
+      <mesh filename="file://$(find sim_description)/meshes/__visual__eye_CAM_1_5a890c16d0_0.stl" scale="0.001 0.001 0.001"/>
+    </geometry>
+    <material name="fusion_Plastic___Glossy__Black__e2e6ed1680"/>
   </visual>
   <collision>
@@ -250,10 +250,10 @@
     <inertia ixx="0.0" iyy="0.0" izz="0.0" ixy="0.0" iyz="-0.0" ixz="0.0"/>
   </inertial>
-  <visual>
+  <visual name="visual_0">
     <origin xyz="-0.27 0.11 -0.21" rpy="0 0 0"/>
     <geometry>
-      <mesh filename="file://$(find sim_description)/meshes/motion_IMU_1.stl" scale="0.001 0.001 0.001"/>
-    </geometry>
-    <material name="silver"/>
+      <mesh filename="file://$(find sim_description)/meshes/__visual__motion_IMU_1_9386f0f59d_0.stl" scale="0.001 0.001 0.001"/>
+    </geometry>
+    <material name="fusion_Steel___Satin_7dcf9b04aa"/>
   </visual>
   <collision>
@@ -328,17 +328,13 @@
   <limit upper="0.523599" lower="0.523599" effort="100" velocity="100"/>
 </joint>
-<joint name="Revolute 34" type="revolute">
+<joint name="Rigid 34" type="fixed">
   <origin xyz="0.072218 -0.03 -0.047303" rpy="0 0 0"/>
   <parent link="Eye-Piece_other_1"/>
   <child link="eye_CAM_1"/>
-  <axis xyz="0.0 -1.0 0.0"/>
-  <limit upper="0.0" lower="0.0" effort="100" velocity="100"/>
-</joint>
-<joint name="Revolute 35" type="revolute">
+</joint>
+<joint name="Rigid 35" type="fixed">
   <origin xyz="0.27 -0.11 0.21" rpy="0 0 0"/>
   <parent link="base_link"/>
   <child link="motion_IMU_1"/>
-  <axis xyz="0.0 0.0 1.0"/>
-  <limit upper="0.0" lower="0.0" effort="100" velocity="100"/>
 </joint>
 </robot>

Commit message: [Sim] FINALLLY figured out some movement controls

File: urdf/materials.xacro (robot description, xacro)
@@ -1,2 +1,2 @@
 <?xml version='1.0' encoding='utf-8'?>
-<robot name="sim" xmlns:xacro="http://www.ros.org/wiki/xacro"><material name="fusion_Nylon_12__with_Formlabs_Fuse_1_3D_Printer__9b6938a61d"><color rgba="0.24705882 0.24705882 0.24705882 1" /></material><material name="fusion_Steel___Satin_7dcf9b04aa"><color rgba="0.62352941 0.62352941 0.62352941 1" /></material><material name="fusion_Plastic___Glossy__Black__77387cc1bc"><color rgba="0.098039216 0.098039216 0.098039216 0" /></material><material name="fusion_Paek__Beige__c3b53efd9f"><color rgba="0.97647059 0.6745098 0.18431373 1" /></material><material name="fusion_Plastic___Glossy__Black__e2e6ed1680"><color rgba="0.098039216 0.098039216 0.098039216 1" /></material></robot>
+<robot name="sim" xmlns:xacro="http://www.ros.org/wiki/xacro"><material name="fusion_Nylon_12__with_Formlabs_Fuse_1_3D_Printer__9b6938a61d"><color rgba="0.24705882 0.24705882 0.24705882 1" /></material><material name="fusion_Steel___Satin_7dcf9b04aa"><color rgba="0.62352941 0.62352941 0.62352941 1" /></material><material name="fusion_Paek__Beige__c3b53efd9f"><color rgba="0.97647059 0.6745098 0.18431373 1" /></material><material name="fusion_Plastic___Glossy__Black__e2e6ed1680"><color rgba="0.098039216 0.098039216 0.098039216 1" /></material></robot>

File: urdf/sim.xacro (robot description, xacro)
@@ -51,5 +51,5 @@
   </inertial>
   <visual name="visual_0">
-    <origin xyz="-0.665 0.042358 -0.017023" rpy="0 0 0"/>
+    <origin xyz="-0.39 0.042358 -0.017023" rpy="0 0 0"/>
     <geometry>
       <mesh filename="file://$(find sim_description)/meshes/__visual__Wheel2_1_6cc1698ccd_0.stl" scale="0.001 0.001 0.001"/>
@@ -58,5 +58,5 @@
   </visual>
   <collision>
-    <origin xyz="-0.665 0.042358 -0.017023" rpy="0 0 0"/>
+    <origin xyz="-0.39 0.042358 -0.017023" rpy="0 0 0"/>
     <geometry>
       <mesh filename="file://$(find sim_description)/meshes/Wheel2_1.stl" scale="0.001 0.001 0.001"/>
@@ -71,5 +71,5 @@
   </inertial>
   <visual name="visual_0">
-    <origin xyz="-0.665 -0.057642 -0.017023" rpy="0 0 0"/>
+    <origin xyz="-0.39 -0.057642 -0.017023" rpy="0 0 0"/>
     <geometry>
       <mesh filename="file://$(find sim_description)/meshes/__visual__Wheels_1_594b391ede_0.stl" scale="0.001 0.001 0.001"/>
@@ -78,5 +78,5 @@
   </visual>
   <collision>
-    <origin xyz="-0.665 -0.057642 -0.017023" rpy="0 0 0"/>
+    <origin xyz="-0.39 -0.057642 -0.017023" rpy="0 0 0"/>
     <geometry>
       <mesh filename="file://$(find sim_description)/meshes/Wheels_1.stl" scale="0.001 0.001 0.001"/>
@@ -91,5 +91,5 @@
   </inertial>
   <visual name="visual_0">
-    <origin xyz="-0.415 0.042358 -0.017023" rpy="0 0 0"/>
+    <origin xyz="-0.143432 0.042358 -0.017023" rpy="0 0 0"/>
     <geometry>
       <mesh filename="file://$(find sim_description)/meshes/__visual__Wheels3_1_788b86b6ca_0.stl" scale="0.001 0.001 0.001"/>
@@ -98,5 +98,5 @@
   </visual>
   <collision>
-    <origin xyz="-0.415 0.042358 -0.017023" rpy="0 0 0"/>
+    <origin xyz="-0.143432 0.042358 -0.017023" rpy="0 0 0"/>
     <geometry>
       <mesh filename="file://$(find sim_description)/meshes/Wheels3_1.stl" scale="0.001 0.001 0.001"/>
@@ -111,5 +111,5 @@
   </inertial>
   <visual name="visual_0">
-    <origin xyz="-0.415 -0.057642 -0.017023" rpy="0 0 0"/>
+    <origin xyz="-0.143432 -0.057642 -0.017023" rpy="0 0 0"/>
     <geometry>
       <mesh filename="file://$(find sim_description)/meshes/__visual__Wheels4_1_2e6ca671c6_0.stl" scale="0.001 0.001 0.001"/>
@@ -118,5 +118,5 @@
   </visual>
   <collision>
-    <origin xyz="-0.415 -0.057642 -0.017023" rpy="0 0 0"/>
+    <origin xyz="-0.143432 -0.057642 -0.017023" rpy="0 0 0"/>
     <geometry>
       <mesh filename="file://$(find sim_description)/meshes/Wheels4_1.stl" scale="0.001 0.001 0.001"/>
@@ -269,29 +269,29 @@
   <child link="Button_Head_Small_Solid_Rivet_ASME_B18.1.1_-_3/8_x_1_1/4_Steel_Plain_1"/>
 </joint>
-<joint name="Revolute 8" type="continuous">
-  <origin xyz="0.665 -0.042358 0.017023" rpy="0 0 0"/>
+<joint name="RF_Whe" type="continuous">
+  <origin xyz="0.39 -0.042358 0.017023" rpy="0 0 0"/>
   <parent link="base_link"/>
   <child link="Wheel2_1"/>
   <axis xyz="1.0 0.0 0.0"/>
 </joint>
-<joint name="Revolute 9" type="continuous">
-  <origin xyz="0.665 0.057642 0.017023" rpy="0 0 0"/>
+<joint name="RB_Whe" type="continuous">
+  <origin xyz="0.39 0.057642 0.017023" rpy="0 0 0"/>
   <parent link="base_link"/>
   <child link="Wheels_1"/>
   <axis xyz="1.0 0.0 0.0"/>
 </joint>
-<joint name="Revolute 10" type="continuous">
-  <origin xyz="0.415 -0.042358 0.017023" rpy="0 0 0"/>
+<joint name="LF_Whe" type="continuous">
+  <origin xyz="0.143432 -0.042358 0.017023" rpy="0 0 0"/>
   <parent link="base_link"/>
   <child link="Wheels3_1"/>
   <axis xyz="-1.0 0.0 0.0"/>
 </joint>
-<joint name="Revolute 11" type="continuous">
-  <origin xyz="0.415 0.057642 0.017023" rpy="0 0 0"/>
+<joint name="LB_Whe" type="continuous">
+  <origin xyz="0.143432 0.057642 0.017023" rpy="0 0 0"/>
   <parent link="base_link"/>
   <child link="Wheels4_1"/>
   <axis xyz="-1.0 0.0 0.0"/>
 </joint>
-<joint name="Revolute 27" type="revolute">
+<joint name="LH" type="revolute">
   <origin xyz="0.158 -0.052358 0.109854" rpy="0 0 0"/>
   <parent link="base_link"/>
@@ -300,5 +300,5 @@
   <limit upper="1.570796" lower="-0.436332" effort="100" velocity="100"/>
 </joint>
-<joint name="Revolute 28" type="revolute">
+<joint name="RH" type="revolute">
   <origin xyz="0.382 -0.052358 0.109854" rpy="0 0 0"/>
   <parent link="base_link"/>
@@ -307,5 +307,5 @@
   <limit upper="0.523599" lower="-1.570796" effort="100" velocity="100"/>
 </joint>
-<joint name="Revolute 29" type="revolute">
+<joint name="Ne" type="revolute">
   <origin xyz="0.27 -0.007358 0.2" rpy="0 0 0"/>
   <parent link="base_link"/>
@@ -314,5 +314,5 @@
   <limit upper="0.698132" lower="-0.698132" effort="100" velocity="100"/>
 </joint>
-<joint name="Revolute 32" type="revolute">
+<joint name="Le" type="revolute">
   <origin xyz="0.0 0.015 0.149854" rpy="0 0 0"/>
   <parent link="Neck_1"/>
@@ -321,5 +321,5 @@
   <limit upper="0.261799" lower="0.261799" effort="100" velocity="100"/>
 </joint>
-<joint name="Revolute 33" type="revolute">
+<joint name="Re" type="revolute">
   <origin xyz="0.0 -0.01 0.0" rpy="0 0 0"/>
   <parent link="Eye-Piece_1"/>
